File: KiCad Schematics/District1.sch (KiCad schematic (older format))
At the start: 24 parts, among them M1 Fan, P2 TERM_08

Commit message: Updated schematic
Added 10A circuit breaker.
Parts:
- added CB1: 10A, symbol FUSE
Connections:
- wire segments 150 -> 151
Other:
- note added: "Connect to TR1 chassis."
- note added: "Panel mounted\ncircuit breaker."
- note added: "To downstream boosters."
Changed lines of the file:
@@
 U 1 1 57C0B9F1
 P 2690 2790
-F 0 "D1" H 2840 3080 50  0000 C CNN
-F 1 "Rectifier" H 2950 3150 50  0000 C CNN
+F 0 "D1" H 2230 3070 50  0000 C CNN
+F 1 "Rectifier" H 2340 3140 50  0000 C CNN
 F 2 "" H 2690 2790 50  0000 C CNN
 F 3 "" H 2690 2790 50  0000 C CNN
@@
 	2360 2000 2360 2150
 Wire Wire Line
-	2360 2150 3110 2150
-Wire Wire Line
-	3110 2150 3110 1250
-Wire Wire Line
-	3110 1250 1550 1250
+	2360 2150 3180 2150
+Wire Wire Line
+	1550 1250 3180 1250
 Wire Wire Line
 	1550 1350 3010 1350
@@
 Wire Bus Line
 	4220 500  4220 1800
-Text Notes 3180 2160 0    60   ~ 0
+Text Notes 2810 2340 0    60   ~ 0
 Primary wired parallel\nSecondary wired in series
 Text Notes 5510 5770 0    60   ~ 0
@@
 Wire Bus Line
 	1070 4820 2020 4820
+Text Notes 1700 1150 0    60   ~ 0
+Connect to TR1 chassis.
+Text Notes 3990 5860 1    60   ~ 0
+To downstream boosters.
+$Comp
+L FUSE CB1
+U 1 1 57C49525
+P 3180 1770
+F 0 "CB1" H 3280 1820 50  0000 C CNN
+F 1 "10A" H 3080 1720 50  0000 C CNN
+F 2 "" H 3180 1770 50  0000 C CNN
+F 3 "" H 3180 1770 50  0000 C CNN
+	1    3180 1770
+	0    1    1    0
+$EndComp
+Wire Wire Line
+	3180 2150 3180 2020
+Wire Wire Line
+	3180 1250 3180 1520
+Text Notes 3290 1940 0    60   ~ 0
+Panel mounted\ncircuit breaker.
 $EndSCHEMATC

Commit message: Schematic updates and printed
More minor changes to the schematic and printed to PDF.
Parts:
- added M?: M-Junction_Box, symbol M-Junction_Box_No-Tap
Connections:
- net labels added: SD_1-3
- net labels removed: SD-1, SD-2, SD-3
- wire segments 151 -> 160
Other:
- note added: "Sub-districts 1-4\ncorrespond to discreet\nyard sections."
- note added: "To 120 VAC\nPower Strip"
- note added: "To downstream\nboosters."
- note removed: "To downstream boosters."
- moved on the sheet: B1, B2, B3, B4
Changed lines of the file:
@@
 $EndComp
 Entry Wire Line
-	9610 3660 9710 3560
-Entry Wire Line
-	9610 3740 9710 3640
-Entry Wire Line
-	9710 3820 9810 3720
-Entry Wire Line
-	9710 3900 9810 3800
+	9810 3660 9910 3560
+Entry Wire Line
+	9810 3740 9910 3640
+Entry Wire Line
+	9810 3820 9910 3720
+Entry Wire Line
+	9810 3900 9910 3800
 Entry Wire Line
 	9810 3980 9910 3880
@@
 	9810 4060 9910 3960
 Entry Wire Line
-	9610 2420 9710 2520
-Entry Wire Line
-	9610 2320 9710 2420
-Entry Wire Line
-	9710 2220 9810 2320
-Entry Wire Line
-	9710 2120 9810 2220
+	9810 2420 9910 2520
+Entry Wire Line
+	9810 2320 9910 2420
+Entry Wire Line
+	9810 2220 9910 2320
+Entry Wire Line
+	9810 2120 9910 2220
 Entry Wire Line
 	9810 2020 9910 2120
 Entry Wire Line
 	9810 1920 9910 2020
-Text Label 9710 3450 1    60   ~ 0
-SD-1
-Text Label 9810 3230 1    60   ~ 0
-SD-2
-Text Label 9910 3010 1    60   ~ 0
-SD-3
+Text Label 9910 3260 1    60   ~ 0
+SD_1-3
 Entry Wire Line
 	9610 4300 9710 4400
@@
 Entry Wire Line
 	9710 4140 9810 4240
-Text Label 9710 5180 1    60   ~ 0
+Text Label 9240 4680 2    60   ~ 0
 DCC-GROUND
-Text Label 9810 4600 1    60   ~ 0
+Text Label 8970 4880 2    60   ~ 0
 16VAC
 Entry Wire Line
@@
 	9510 2020 9810 2020
 Wire Wire Line
-	9510 2120 9710 2120
-Wire Wire Line
-	9510 2220 9710 2220
-Wire Wire Line
-	9510 2320 9610 2320
-Wire Wire Line
-	9510 2420 9610 2420
-Wire Wire Line
-	9510 3660 9610 3660
-Wire Wire Line
-	9510 3740 9610 3740
-Wire Wire Line
-	9510 3820 9710 3820
-Wire Wire Line
-	9510 3900 9710 3900
+	9510 2120 9810 2120
+Wire Wire Line
+	9510 2220 9810 2220
+Wire Wire Line
+	9510 2320 9810 2320
+Wire Wire Line
+	9510 2420 9810 2420
+Wire Wire Line
+	9510 3660 9810 3660
+Wire Wire Line
+	9510 3740 9810 3740
+Wire Wire Line
+	9510 3820 9810 3820
+Wire Wire Line
+	9510 3900 9810 3900
 Wire Wire Line
 	9510 3980 9810 3980
 Wire Wire Line
 	9510 4060 9810 4060
-Wire Bus Line
-	9710 2420 9710 3640
-Wire Bus Line
-	9810 2220 9810 3800
-Wire Bus Line
-	9910 2020 9910 3960
 Wire Wire Line
 	9510 4300 9610 4300
@@
 Wire Wire Line
 	9510 4140 9710 4140
-Wire Bus Line
-	9710 4400 9710 5190
-Wire Bus Line
-	9810 4240 9810 5190
 Wire Bus Line
 	9690 910  9690 1720
@@
 Text Notes 2810 2340 0    60   ~ 0
 Primary wired parallel\nSecondary wired in series
-Text Notes 5510 5770 0    60   ~ 0
-To 120 VAC Power Strip
+Text Notes 5510 5910 0    60   ~ 0
+To 120 VAC\nPower Strip
 Wire Bus Line
 	4940 5370 5460 5370
@@
 L Crystal B2
 U 1 1 57C2E519
-P 8350 5110
-F 0 "B2" H 8350 5260 50  0000 C CNN
-F 1 "Piezo" H 8350 4960 50  0000 C CNN
-F 2 "" H 8350 5110 50  0000 C CNN
-F 3 "" H 8350 5110 50  0000 C CNN
-	1    8350 5110
+P 7470 5110
+F 0 "B2" H 7470 5260 50  0000 C CNN
+F 1 "Piezo" H 7470 4960 50  0000 C CNN
+F 2 "" H 7470 5110 50  0000 C CNN
+F 3 "" H 7470 5110 50  0000 C CNN
+	1    7470 5110
 	1    0    0    -1
 $EndComp
@@
 L Crystal B3
 U 1 1 57C2E622
-P 8350 5490
-F 0 "B3" H 8350 5640 50  0000 C CNN
-F 1 "Piezo" H 8350 5340 50  0000 C CNN
-F 2 "" H 8350 5490 50  0000 C CNN
-F 3 "" H 8350 5490 50  0000 C CNN
-	1    8350 5490
+P 7470 5490
+F 0 "B3" H 7470 5640 50  0000 C CNN
+F 1 "Piezo" H 7470 5340 50  0000 C CNN
+F 2 "" H 7470 5490 50  0000 C CNN
+F 3 "" H 7470 5490 50  0000 C CNN
+	1    7470 5490
 	1    0    0    -1
 $EndComp
@@
 L Crystal B4
 U 1 1 57C2E6BB
-P 8350 5860
-F 0 "B4" H 8350 6010 50  0000 C CNN
-F 1 "Piezo" H 8350 5710 50  0000 C CNN
-F 2 "" H 8350 5860 50  0000 C CNN
-F 3 "" H 8350 5860 50  0000 C CNN
-	1    8350 5860
+P 7470 5860
+F 0 "B4" H 7470 6010 50  0000 C CNN
+F 1 "Piezo" H 7470 5710 50  0000 C CNN
+F 2 "" H 7470 5860 50  0000 C CNN
+F 3 "" H 7470 5860 50  0000 C CNN
+	1    7470 5860
 	1    0    0    -1
 $EndComp
@@
 L Crystal B1
 U 1 1 57C2E788
-P 8350 4730
-F 0 "B1" H 8350 4880 50  0000 C CNN
-F 1 "Piezo" H 8350 4580 50  0000 C CNN
-F 2 "" H 8350 4730 50  0000 C CNN
-F 3 "" H 8350 4730 50  0000 C CNN
-	1    8350 4730
+P 7470 4730
+F 0 "B1" H 7470 4880 50  0000 C CNN
+F 1 "Piezo" H 7470 4580 50  0000 C CNN
+F 2 "" H 7470 4730 50  0000 C CNN
+F 3 "" H 7470 4730 50  0000 C CNN
+	1    7470 4730
 	1    0    0    -1
 $EndComp
 Wire Wire Line
-	8500 4730 8600 4730
-Entry Wire Line
-	8600 4730 8700 4830
-Wire Wire Line
-	8500 5110 8600 5110
-Wire Wire Line
-	8500 5490 8600 5490
-Wire Wire Line
-	8500 5860 8600 5860
-Entry Wire Line
-	8600 5110 8700 5210
-Entry Wire Line
-	8600 5490 8700 5590
-Entry Wire Line
-	8600 5860 8700 5960
-Entry Wire Line
-	8000 5760 8100 5860
-Wire Wire Line
-	8200 5860 8100 5860
-Wire Wire Line
-	8200 5490 8100 5490
-Wire Wire Line
-	8200 5110 8100 5110
-Wire Wire Line
-	8200 4730 8100 4730
-Entry Wire Line
-	8000 5390 8100 5490
-Entry Wire Line
-	8000 5010 8100 5110
-Entry Wire Line
-	8000 4630 8100 4730
-Wire Bus Line
-	8000 3250 8000 6200
-Wire Bus Line
-	8700 4830 8700 6200
-Wire Bus Line
-	8700 6200 8000 6200
+	7620 4730 7720 4730
+Entry Wire Line
+	7720 4730 7820 4830
+Wire Wire Line
+	7620 5110 7720 5110
+Wire Wire Line
+	7620 5490 7720 5490
+Wire Wire Line
+	7620 5860 7720 5860
+Entry Wire Line
+	7720 5110 7820 5210
+Entry Wire Line
+	7720 5490 7820 5590
+Entry Wire Line
+	7720 5860 7820 5960
+Entry Wire Line
+	7120 5760 7220 5860
+Wire Wire Line
+	7320 5860 7220 5860
+Wire Wire Line
+	7320 5490 7220 5490
+Wire Wire Line
+	7320 5110 7220 5110
+Wire Wire Line
+	7320 4730 7220 4730
+Entry Wire Line
+	7120 5390 7220 5490
+Entry Wire Line
+	7120 5010 7220 5110
+Entry Wire Line
+	7120 4630 7220 4730
+Wire Bus Line
+	7120 3250 7120 6200
+Wire Bus Line
+	7820 4830 7820 6200
+Wire Bus Line
+	7820 6200 7120 6200
 Wire Wire Line
 	8290 2220 8390 2220
@@
 	8490 2320 8490 3250
 Wire Bus Line
-	8490 3250 8000 3250
+	8490 3250 7120 3250
 Text Label 8490 2900 1    60   ~ 0
 Alarm-Bus
@@
 Text Notes 1700 1150 0    60   ~ 0
 Connect to TR1 chassis.
-Text Notes 3990 5860 1    60   ~ 0
-To downstream boosters.
+Text Notes 3700 5460 0    60   ~ 0
+To downstream\nboosters.
 $Comp
 L FUSE CB1
@@
 Text Notes 3290 1940 0    60   ~ 0
 Panel mounted\ncircuit breaker.
+$Comp
+L M-Junction_Box_No-Tap M?
+U 1 1 57C4EDF8
+P 8610 5200
+F 0 "M?" H 8680 5040 60  0001 C CNN
+F 1 "M-Junction_Box" H 8620 5120 60  0000 L CNN
+F 2 "" H 8610 5200 60  0000 C CNN
+F 3 "" H 8610 5200 60  0000 C CNN
+	1    8610 5200
+	1    0    0    1
+$EndComp
+Entry Wire Line
+	9810 5250 9910 5150
+Entry Wire Line
+	9810 5330 9910 5230
+Entry Wire Line
+	9810 5410 9910 5310
+Entry Wire Line
+	9810 5490 9910 5390
+Entry Wire Line
+	9810 5570 9910 5470
+Entry Wire Line
+	9810 5650 9910 5550
+Wire Wire Line
+	9510 5250 9810 5250
+Wire Wire Line
+	9510 5330 9810 5330
+Wire Wire Line
+	9510 5410 9810 5410
+Wire Wire Line
+	9510 5490 9810 5490
+Wire Wire Line
+	9510 5570 9810 5570
+Wire Wire Line
+	9510 5650 9810 5650
+Entry Wire Line
+	9610 5890 9710 5990
+Entry Wire Line
+	9710 5810 9810 5910
+Entry Wire Line
+	9710 5730 9810 5830
+Wire Wire Line
+	9510 5890 9610 5890
+Wire Wire Line
+	9510 5810 9710 5810
+Wire Wire Line
+	9510 5730 9710 5730
+Wire Bus Line
+	9710 4400 9710 4680
+Wire Bus Line
+	9710 4680 8600 4680
+Wire Bus Line
+	9810 4240 9810 4880
+Wire Bus Line
+	9810 4880 8600 4880
+Text Label 9240 6270 2    60   ~ 0
+DCC-GROUND
+Text Label 8970 6470 2    60   ~ 0
+16VAC
+Wire Bus Line
+	9710 5990 9710 6270
+Wire Bus Line
+	9710 6270 8600 6270
+Wire Bus Line
+	9810 5830 9810 6470
+Wire Bus Line
+	9810 6470 8600 6470
+Wire Bus Line
+	9910 2020 9910 5550
+Text Notes 8820 2870 0    60   ~ 0
+Sub-districts 1-4\ncorrespond to discreet\nyard sections.
 $EndSCHEMATC

Commit message: Updated schematics
Fixed wiring using the correct pin-outs for the Triad transformers. Made
other minor changes.
Parts:
- removed TR1: 16VCT, symbol TRANSFORMER_MCI_4-49-8016
- added TR1: VPS16, symbol TRANSFORMER_VPS16
Changed lines of the file:
@@
 $Descr USLetter 11000 8500
 encoding utf-8
-Sheet 2 3
+Sheet 2 4
 Title "District 1 Power Box"
 Date "2016-08-27"
-Rev ""
+Rev "2"
 Comp "North Georgia Modurail"
 Comment1 ""
@@
 $EndComp
 $Comp
-L TRANSFORMER_MCI_4-49-8016 TR1
-U 1 1 57C0B936
-P 2620 1830
-F 0 "TR1" V 2620 2270 50  0000 C CNN
-F 1 "16VCT" V 2550 2220 50  0000 C CNN
-F 2 "" H 2620 1830 60  0000 C CNN
-F 3 "" H 2620 1830 60  0000 C CNN
-	1    2620 1830
-	0    -1   -1   0
-$EndComp
-$Comp
 L Diode_Bridge D1
 U 1 1 57C0B9F1
@@
 Wire Wire Line
 	1550 1450 2910 1450
-Wire Wire Line
-	1550 1550 2710 1550
 Connection ~ 2080 1550
 Wire Wire Line
@@
 	9690 910  9690 1720
 Wire Wire Line
-	2360 1550 2360 1660
-Wire Wire Line
-	2560 1450 2560 1660
-Wire Wire Line
-	2710 1550 2710 1660
-Connection ~ 2360 1550
-Wire Wire Line
 	2910 1450 2910 1660
-Connection ~ 2560 1450
-Wire Wire Line
-	2560 2000 2560 2100
-Wire Wire Line
-	2560 2100 2710 2100
-Wire Wire Line
-	2710 2100 2710 2000
 Wire Wire Line
 	2360 2000 2360 2150
@@
 Wire Wire Line
 	1550 1350 3010 1350
-Wire Wire Line
-	3010 1350 3010 2100
-Wire Wire Line
-	3010 2100 2910 2100
-Wire Wire Line
-	2910 2100 2910 2000
 Wire Wire Line
 	1550 1150 3290 1150
@@
 U 1 1 57C49525
 P 3180 1770
-F 0 "CB1" H 3280 1820 50  0000 C CNN
-F 1 "10A" H 3080 1720 50  0000 C CNN
+F 0 "CB1" V 3290 1860 50  0000 C CNN
+F 1 "10A" V 3360 1860 50  0000 C CNN
 F 2 "" H 3180 1770 50  0000 C CNN
 F 3 "" H 3180 1770 50  0000 C CNN
@@
 Wire Wire Line
 	3180 1250 3180 1520
-Text Notes 3290 1940 0    60   ~ 0
+Text Notes 3290 1840 0    60   ~ 0
 Panel mounted\ncircuit breaker.
 $Comp
@@
 Text Notes 8820 2870 0    60   ~ 0
 Sub-districts 1-4\ncorrespond to discreet\nyard sections.
+$Comp
+L TRANSFORMER_VPS16 TR1
+U 1 1 57E17910
+P 2620 1830
+F 0 "TR1" V 2620 2210 50  0000 C CNN
+F 1 "VPS16" V 2550 2230 50  0000 C CNN
+F 2 "" H 2620 1830 60  0000 C CNN
+F 3 "" H 2620 1830 60  0000 C CNN
+	1    2620 1830
+	0    -1   -1   0
+$EndComp
+Wire Wire Line
+	2710 2000 2710 2150
+Connection ~ 2710 2150
+Wire Wire Line
+	3010 1350 3010 2070
+Wire Wire Line
+	3010 2070 2560 2070
+Wire Wire Line
+	2560 2070 2560 2000
+Wire Wire Line
+	2910 2000 2910 2070
+Connection ~ 2910 2070
+Wire Wire Line
+	1550 1550 2360 1550
+Wire Wire Line
+	2360 1550 2360 1660
+Wire Wire Line
+	2560 1660 2560 1550
+Wire Wire Line
+	2560 1550 2710 1550
+Wire Wire Line
+	2710 1550 2710 1660
 $EndSCHEMATC

Commit message: Updated schematic
Parts:
- TR1: symbol TRANSFORMER_VPS16 -> TRANSFORMER_VPS16-RESCUE-NGM_Power_Box
Changed lines of the file:
@@
 $Descr USLetter 11000 8500
 encoding utf-8
-Sheet 2 6
+Sheet 2 7
 Title "District 1 Power Box"
 Date "2016-09-30"
@@
 Sub-districts 1-4\ncorrespond to discreet\nyard sections.
 $Comp
-L TRANSFORMER_VPS16 TR1
+L TRANSFORMER_VPS16-RESCUE-NGM_Power_Box TR1
 U 1 1 57E17910
 P 2620 1830
