File: KiCad Schematics/Remote-District.sch (KiCad schematic (older format))
At the start: 17 parts, among them M1 Fan

Commit message: Updated schematic
Added 10A circuit breaker.
Other:
- note added: "Connect to TR1 chassis."
- note added: "From upstream LNRP"
Changed lines of the file:
@@
 Wire Bus Line
 	7590 5130 7590 2220
+Wire Bus Line
+	2030 5550 560  5550
+Wire Bus Line
+	560  5550 560  7160
+Wire Bus Line
+	560  7160 3490 7160
+Text Label 1620 7170 0    60   ~ 0
+Protected_LocoNet
+Text Notes 2020 7290 0    60   ~ 0
+From upstream LNRP
+Text Notes 1520 1150 0    60   ~ 0
+Connect to TR1 chassis.
 $EndSCHEMATC

Commit message: Schematic updates and printed
More minor changes to the schematic and printed to PDF.
Parts:
- added CB1: 10A, symbol FUSE
- added M?: M-Junction_Box, symbol M-Junction_Box_No-Tap
Connections:
- net labels added: SD_1-3
- net labels removed: SD-1, SD-2, SD-3
- wire segments 109 -> 119
Other:
- note added: "Panel mounted\ncircuit breaker."
- note added: "Sub-districts 1-3\ncorrespond to\ntracks 1-3."
- note added: "To 120 VAC\nPower Strip"
- note added: "To downstream\nboosters"
- note removed: "Sub-districts 1-3 correspond to tracks 1-3"
- note removed: "To 120VAC Power Strip"
- note removed: "To downstream boosters"
Changed lines of the file:
@@
 	1550 1350 2070 1350
 Wire Wire Line
-	1550 1450 2900 1450
+	1550 1450 3010 1450
 Wire Wire Line
 	1550 1550 2820 1550
@@
 PS14
 Wire Bus Line
-	4360 5500 3870 5500
-Wire Bus Line
-	3870 5500 3870 4810
+	3870 5500 4360 5500
+Wire Bus Line
+	3870 4590 3870 5500
 Text Label 3870 5410 1    60   ~ 0
 Protected_LocoNet
@@
 Entry Wire Line
 	4940 4520 5040 4420
-Text Label 5170 4420 2    60   ~ 0
+Text Label 5310 3590 3    60   ~ 0
 Standard_LocoNet
 Wire Wire Line
@@
 	9510 2020 9810 2020
 Wire Wire Line
-	9510 2120 9710 2120
-Wire Wire Line
-	9510 2220 9710 2220
-Wire Wire Line
-	9510 2320 9610 2320
-Wire Wire Line
-	9510 2420 9610 2420
+	9510 2120 9810 2120
+Wire Wire Line
+	9510 2220 9810 2220
+Wire Wire Line
+	9510 2320 9810 2320
+Wire Wire Line
+	9510 2420 9810 2420
 $Comp
 L M-Junction_Box_No-Tap M?
@@
 $EndComp
 Wire Wire Line
-	9510 3660 9610 3660
-Wire Wire Line
-	9510 3740 9610 3740
-Wire Wire Line
-	9510 3820 9710 3820
-Wire Wire Line
-	9510 3900 9710 3900
+	9510 3660 9810 3660
+Wire Wire Line
+	9510 3740 9810 3740
+Wire Wire Line
+	9510 3820 9810 3820
+Wire Wire Line
+	9510 3900 9810 3900
 Wire Wire Line
 	9510 3980 9810 3980
@@
 	9510 4060 9810 4060
 Entry Wire Line
-	9610 3660 9710 3560
-Entry Wire Line
-	9610 3740 9710 3640
-Entry Wire Line
-	9710 3820 9810 3720
-Entry Wire Line
-	9710 3900 9810 3800
+	9810 3660 9910 3560
+Entry Wire Line
+	9810 3740 9910 3640
+Entry Wire Line
+	9810 3820 9910 3720
+Entry Wire Line
+	9810 3900 9910 3800
 Entry Wire Line
 	9810 3980 9910 3880
@@
 	9810 4060 9910 3960
 Entry Wire Line
-	9610 2420 9710 2520
-Entry Wire Line
-	9610 2320 9710 2420
-Entry Wire Line
-	9710 2220 9810 2320
-Entry Wire Line
-	9710 2120 9810 2220
+	9810 2420 9910 2520
+Entry Wire Line
+	9810 2320 9910 2420
+Entry Wire Line
+	9810 2220 9910 2320
+Entry Wire Line
+	9810 2120 9910 2220
 Entry Wire Line
 	9810 2020 9910 2120
@@
 	9810 1920 9910 2020
 Wire Bus Line
-	9710 2420 9710 3640
-Wire Bus Line
-	9810 2220 9810 3800
-Wire Bus Line
-	9910 2020 9910 3960
-Text Label 9710 3450 1    60   ~ 0
-SD-1
-Text Label 9810 3230 1    60   ~ 0
-SD-2
-Text Label 9910 3010 1    60   ~ 0
-SD-3
+	9910 2020 9910 5550
+Text Label 9910 3310 1    60   ~ 0
+SD_1-3
 Wire Wire Line
 	9510 4300 9610 4300
@@
 Entry Wire Line
 	9710 4140 9810 4240
-Wire Bus Line
-	9710 4400 9710 5190
-Text Label 9710 5180 1    60   ~ 0
+Text Label 8500 6210 2    60   ~ 0
 DCC-GROUND
-Wire Bus Line
-	9810 4240 9810 5190
-Text Label 9810 4600 1    60   ~ 0
+Text Label 8480 6510 2    60   ~ 0
 16VAC
 $Comp
@@
 	2820 1710 2730 1710
 Wire Wire Line
-	2900 1450 2900 2260
-Wire Wire Line
-	2900 2260 2730 2260
+	2730 2260 3010 2260
 Wire Wire Line
 	2070 2260 2390 2260
@@
 Wire Bus Line
 	880  2210 880  3210
-Text Notes 980  600  0    60   ~ 0
-To 120VAC Power Strip
-Text Notes 10180 4100 1    60   ~ 0
-Sub-districts 1-3 correspond to tracks 1-3
+Text Notes 1090 670  0    60   ~ 0
+To 120 VAC\nPower Strip
+Text Notes 8960 2920 0    60   ~ 0
+Sub-districts 1-3\ncorrespond to\ntracks 1-3.
 Wire Wire Line
 	1550 1250 2210 1250
@@
 	2560 1150 2560 1290
 Wire Bus Line
-	4940 4420 5310 4420
-Wire Bus Line
-	5310 4420 5310 3850
+	5310 4420 4940 4420
+Wire Bus Line
+	5310 3590 5310 4420
 Text Notes 4580 4300 0    60   ~ 0
 To local UP5s
-Text Notes 3980 5090 1    60   ~ 0
-To downstream boosters
+Text Notes 3630 4510 0    60   ~ 0
+To downstream\nboosters
 Entry Wire Line
 	5620 2120 5720 2220
@@
 Text Notes 1520 1150 0    60   ~ 0
 Connect to TR1 chassis.
+$Comp
+L FUSE CB1
+U 1 1 57C4A4E5
+P 3010 1890
+F 0 "CB1" H 3110 1940 50  0000 C CNN
+F 1 "10A" H 2910 1840 50  0000 C CNN
+F 2 "" H 3010 1890 50  0000 C CNN
+F 3 "" H 3010 1890 50  0000 C CNN
+	1    3010 1890
+	0    1    1    0
+$EndComp
+Wire Wire Line
+	3010 2260 3010 2140
+Wire Wire Line
+	3010 1450 3010 1640
+Text Notes 3060 1740 0    60   ~ 0
+Panel mounted\ncircuit breaker.
+$Comp
+L M-Junction_Box_No-Tap M?
+U 1 1 57C4B598
+P 8610 5200
+F 0 "M?" H 8680 5040 60  0001 C CNN
+F 1 "M-Junction_Box" H 8620 5120 60  0000 L CNN
+F 2 "" H 8610 5200 60  0000 C CNN
+F 3 "" H 8610 5200 60  0000 C CNN
+	1    8610 5200
+	1    0    0    1
+$EndComp
+Entry Wire Line
+	9810 5250 9910 5150
+Wire Wire Line
+	9510 5250 9810 5250
+Entry Wire Line
+	9810 5330 9910 5230
+Wire Wire Line
+	9510 5330 9810 5330
+Wire Wire Line
+	9510 5410 9810 5410
+Wire Wire Line
+	9510 5490 9810 5490
+Wire Wire Line
+	9510 5570 9810 5570
+Wire Wire Line
+	9510 5650 9810 5650
+Entry Wire Line
+	9810 5410 9910 5310
+Entry Wire Line
+	9810 5490 9910 5390
+Entry Wire Line
+	9810 5570 9910 5470
+Entry Wire Line
+	9810 5650 9910 5550
+Wire Wire Line
+	9510 5890 9610 5890
+Wire Wire Line
+	9510 5810 9710 5810
+Wire Wire Line
+	9510 5730 9710 5730
+Entry Wire Line
+	9610 5890 9710 5990
+Entry Wire Line
+	9710 5810 9810 5910
+Entry Wire Line
+	9710 5730 9810 5830
+Wire Bus Line
+	9810 4240 9810 4960
+Wire Bus Line
+	9810 4960 8170 4960
+Wire Bus Line
+	9710 4400 9710 4670
+Wire Bus Line
+	9710 4670 7980 4670
+Wire Bus Line
+	9710 5990 9710 6210
+Wire Bus Line
+	9710 6210 7790 6210
+Wire Bus Line
+	9810 5830 9810 6510
+Wire Bus Line
+	9810 6510 7780 6510
+Text Label 8780 4670 2    60   ~ 0
+DCC-GROUND
+Text Label 9000 4960 2    60   ~ 0
+16VAC
+Text Notes 5470 4960 0    60   ~ 0
+To 120 VAC\nPower Strip
 $EndSCHEMATC

Commit message: Update schematic
Parts:
- added 2A: CB2, symbol FUSE
Connections:
- wire segments 119 -> 123
Changed lines of the file:
@@
 	5160 3530 4520 3530
 Wire Bus Line
-	1320 6410 3530 6410
+	3530 6410 1320 6410
 Wire Wire Line
 	3740 3430 3630 3430
@@
 Entry Wire Line
 	9710 4140 9810 4240
-Text Label 8500 6210 2    60   ~ 0
+Text Label 9050 6210 2    60   ~ 0
 DCC-GROUND
-Text Label 8480 6510 2    60   ~ 0
+Text Label 8560 6510 2    60   ~ 0
 16VAC
 $Comp
@@
 	3420 570  3420 1250
 Wire Bus Line
-	3530 6410 3530 3530
+	3530 3530 3530 6410
 Wire Bus Line
 	550  1550 550  4690
@@
 	2560 1150 2560 1290
 Wire Bus Line
-	5310 4420 4940 4420
-Wire Bus Line
-	5310 3590 5310 4420
+	4940 4420 5310 4420
+Wire Bus Line
+	5310 4420 5310 3590
 Text Notes 4580 4300 0    60   ~ 0
 To local UP5s
@@
 	6890 4140 6890 5130
 Wire Bus Line
-	6890 5130 7590 5130
-Wire Bus Line
-	7590 5130 7590 2220
-Wire Bus Line
-	2030 5550 560  5550
-Wire Bus Line
-	560  5550 560  7160
-Wire Bus Line
-	560  7160 3490 7160
+	7590 5130 6890 5130
+Wire Bus Line
+	7590 2220 7590 5130
+Wire Bus Line
+	2030 5550 1140 5550
+Wire Bus Line
+	1140 5550 1140 7160
+Wire Bus Line
+	1140 7160 3490 7160
 Text Label 1620 7170 0    60   ~ 0
 Protected_LocoNet
@@
 	9710 5990 9710 6210
 Wire Bus Line
-	9710 6210 7790 6210
-Wire Bus Line
-	9810 5830 9810 6510
-Wire Bus Line
-	9810 6510 7780 6510
+	9710 6210 8370 6210
+Wire Bus Line
+	9810 6510 9810 5830
+Wire Bus Line
+	7780 6510 9810 6510
 Text Label 8780 4670 2    60   ~ 0
 DCC-GROUND
@@
 Text Notes 5470 4960 0    60   ~ 0
 To 120 VAC\nPower Strip
+$Comp
+L FUSE 2A
+U 1 1 57C5832F
+P 6840 6410
+F 0 "2A" H 6940 6460 50  0000 C CNN
+F 1 "CB2" H 6740 6360 50  0000 C CNN
+F 2 "" H 6840 6410 50  0000 C CNN
+F 3 "" H 6840 6410 50  0000 C CNN
+	1    6840 6410
+	1    0    0    -1
+$EndComp
+Entry Wire Line
+	7780 6410 7880 6510
+Entry Wire Line
+	7680 6410 7780 6510
+Wire Wire Line
+	7780 6410 7780 6200
+Wire Wire Line
+	7780 6200 6010 6200
+Wire Wire Line
+	7090 6410 7680 6410
+Wire Wire Line
+	6590 6410 6010 6410
+Entry Wire Line
+	5910 6510 6010 6410
+Entry Wire Line
+	5910 6300 6010 6200
+Wire Bus Line
+	5910 6300 5910 7810
+Text Label 5910 6800 3    60   ~ 0
+16VAC
+Text Notes 6560 6680 0    60   ~ 0
+Panel mounted\ncircuit breaker.
+Wire Bus Line
+	8170 4960 8170 6510
+Connection ~ 8170 6510
+Wire Bus Line
+	5910 7810 550  7810
+Wire Bus Line
+	550  7810 550  4680
 $EndSCHEMATC

Commit message: Updated schematics
Fixed wiring using the correct pin-outs for the Triad transformers. Made
other minor changes.
Parts:
- removed TB1: TERM_08, symbol TERM_08
- removed TR1: 16VCT, symbol TRANSFORMER_MCI_4-49-8016
- added TB1: TERM_06, symbol TERM_06
- added TR1: VPS16, symbol TRANSFORMER_VPS16
Connections:
- net labels removed: Earth
- wire segments 123 -> 117
- no-connect marks 8 -> 10
Other:
- note removed: "Connect to TR1 chassis."
- moved on the sheet: CB1, M1
Changed lines of the file:
@@
 $Descr USLetter 11000 8500
 encoding utf-8
-Sheet 3 3
+Sheet 3 4
 Title "District 1 Power Box"
 Date "2016-08-27"
-Rev ""
+Rev "2"
 Comp "North Georgia Modurail"
 Comment1 ""
@@
 	0    1    -1   0
 $EndComp
-$Comp
-L TERM_08 TB1
-U 1 1 57C1C741
-P 1300 1300
-F 0 "TB1" H 1300 1750 50  0000 C CNN
-F 1 "TERM_08" H 1320 850 50  0000 C CNN
-F 2 "" H 1300 100 50  0000 C CNN
-F 3 "" H 1300 100 50  0000 C CNN
-	1    1300 1300
-	1    0    0    -1
-$EndComp
-Entry Wire Line
-	550  1250 650  1350
-Entry Wire Line
-	550  1150 650  1250
-Entry Wire Line
-	550  1050 650  1150
-Entry Wire Line
-	750  950  850  1050
-Entry Wire Line
-	750  850  850  950
-Text Label 750  750  0    60   ~ 0
+Entry Wire Line
+	750  1150 850  1250
+Entry Wire Line
+	750  1050 850  1150
+Text Label 750  950  0    60   ~ 0
 12VDC
-Text Label 550  600  0    60   ~ 0
+Text Label 2680 670  0    60   ~ 0
 120VAC
 $Comp
 L Fan M1
 U 1 1 57C1C742
-P 2700 850
-F 0 "M1" V 2990 1310 60  0000 C CNN
-F 1 "Fan" V 2900 1250 60  0000 L CNN
-F 2 "" H 2700 850 60  0000 C CNN
-F 3 "" H 2700 850 60  0000 C CNN
-	1    2700 850
+P 1990 1050
+F 0 "M1" V 2280 1510 60  0000 C CNN
+F 1 "Fan" V 2190 1450 60  0000 L CNN
+F 2 "" H 1990 1050 60  0000 C CNN
+F 3 "" H 1990 1050 60  0000 C CNN
+	1    1990 1050
 	0    1    1    0
-$EndComp
-$Comp
-L Earth #PWR?
-U 1 1 57C1C743
-P 2560 1290
-F 0 "#PWR?" H 2560 1040 50  0001 C CNN
-F 1 "Earth" H 2560 1140 50  0001 C CNN
-F 2 "" H 2560 1290 50  0000 C CNN
-F 3 "" H 2560 1290 50  0000 C CNN
-	1    2560 1290
-	1    0    0    -1
 $EndComp
 Entry Wire Line
@@
 	3530 3630 3630 3530
 Wire Wire Line
-	1050 950  850  950
-Wire Wire Line
-	1050 1150 650  1150
-Wire Wire Line
-	1050 1250 650  1250
-Wire Wire Line
-	1050 1350 650  1350
-Wire Bus Line
-	550  600  550  1250
-Wire Wire Line
-	1050 1050 850  1050
-Wire Bus Line
-	750  650  750  950
-Wire Wire Line
-	1550 950  2500 950
-Wire Wire Line
-	1550 1050 2500 1050
-Wire Wire Line
-	1550 1350 2070 1350
-Wire Wire Line
-	1550 1450 3010 1450
-Wire Wire Line
-	1550 1550 2820 1550
+	1050 1150 850  1150
+Wire Wire Line
+	1050 1250 850  1250
+Wire Bus Line
+	750  850  750  1150
 Wire Wire Line
 	1050 1450 650  1450
@@
 	5160 3530 4520 3530
 Wire Bus Line
-	3530 6410 1320 6410
+	1320 6410 3530 6410
 Wire Wire Line
 	3740 3430 3630 3430
@@
 	3420 570  3420 1250
 Wire Bus Line
-	3530 3530 3530 6410
+	3530 6410 3530 3530
 Wire Bus Line
 	550  1550 550  4690
 Wire Wire Line
 	1800 1650 1800 5090
-$Comp
-L TRANSFORMER_MCI_4-49-8016 TR1
-U 1 1 57C213DC
-P 2560 1970
-F 0 "TR1" H 2560 2280 50  0000 C CNN
-F 1 "16VCT" H 2560 1570 50  0000 C CNN
-F 2 "" H 2560 1970 60  0000 C CNN
-F 3 "" H 2560 1970 60  0000 C CNN
-	1    2560 1970
-	1    0    0    -1
-$EndComp
-Wire Wire Line
-	2730 1910 2830 1910
-Wire Wire Line
-	2830 1910 2830 2060
-Wire Wire Line
-	2830 2060 2730 2060
-Wire Wire Line
-	2820 1550 2820 1710
-Wire Wire Line
-	2820 1710 2730 1710
-Wire Wire Line
-	2730 2260 3010 2260
-Wire Wire Line
-	2070 2260 2390 2260
-Wire Wire Line
-	2070 1350 2070 2260
-Wire Wire Line
-	2390 1910 2070 1910
-Connection ~ 2070 1910
-Wire Wire Line
-	2210 2060 2390 2060
-Wire Wire Line
-	2210 1250 2210 2060
-Wire Wire Line
-	2210 1710 2390 1710
-Connection ~ 2210 1710
-Text Notes 1990 2610 0    60   ~ 0
+Wire Wire Line
+	2820 2000 2730 2000
+Wire Wire Line
+	2730 2550 3010 2550
+Text Notes 1990 2900 0    60   ~ 0
 Primary wired parallel\nSecondary wired in series
 Wire Bus Line
 	880  2210 880  3210
-Text Notes 1090 670  0    60   ~ 0
+Text Notes 1470 750  0    60   ~ 0
 To 120 VAC\nPower Strip
 Text Notes 8960 2920 0    60   ~ 0
 Sub-districts 1-3\ncorrespond to\ntracks 1-3.
-Wire Wire Line
-	1550 1250 2210 1250
-Wire Wire Line
-	1550 1150 2560 1150
-Wire Wire Line
-	2560 1150 2560 1290
 Wire Bus Line
 	4940 4420 5310 4420
@@
 	6890 4140 6890 5130
 Wire Bus Line
-	7590 5130 6890 5130
-Wire Bus Line
-	7590 2220 7590 5130
+	6890 5130 7590 5130
+Wire Bus Line
+	7590 5130 7590 2220
 Wire Bus Line
 	2030 5550 1140 5550
@@
 Text Notes 2020 7290 0    60   ~ 0
 From upstream LNRP
-Text Notes 1520 1150 0    60   ~ 0
-Connect to TR1 chassis.
 $Comp
 L FUSE CB1
 U 1 1 57C4A4E5
-P 3010 1890
-F 0 "CB1" H 3110 1940 50  0000 C CNN
-F 1 "10A" H 2910 1840 50  0000 C CNN
-F 2 "" H 3010 1890 50  0000 C CNN
-F 3 "" H 3010 1890 50  0000 C CNN
-	1    3010 1890
+P 3010 2180
+F 0 "CB1" V 3010 2330 50  0000 C CNN
+F 1 "10A" V 3080 2330 50  0000 C CNN
+F 2 "" H 3010 2180 50  0000 C CNN
+F 3 "" H 3010 2180 50  0000 C CNN
+	1    3010 2180
 	0    1    1    0
 $EndComp
 Wire Wire Line
-	3010 2260 3010 2140
-Wire Wire Line
-	3010 1450 3010 1640
-Text Notes 3060 1740 0    60   ~ 0
+	3010 2550 3010 2430
+Text Notes 3060 2030 0    60   ~ 0
 Panel mounted\ncircuit breaker.
 $Comp
@@
 Wire Bus Line
 	550  7810 550  4680
+$Comp
+L TRANSFORMER_VPS16 TR1
+U 1 1 57E184F7
+P 2560 2260
+F 0 "TR1" H 2560 2570 50  0000 C CNN
+F 1 "VPS16" H 2560 1860 50  0000 C CNN
+F 2 "" H 2560 2260 60  0000 C CNN
+F 3 "" H 2560 2260 60  0000 C CNN
+	1    2560 2260
+	-1   0    0    -1
+$EndComp
+Wire Wire Line
+	2820 2350 2730 2350
+Connection ~ 2820 2000
+Wire Wire Line
+	2730 2200 2880 2200
+Wire Wire Line
+	2880 2200 2880 2550
+Connection ~ 2880 2550
+Wire Wire Line
+	2390 2350 2340 2350
+Wire Wire Line
+	2340 2350 2340 2200
+Wire Wire Line
+	2340 2200 2390 2200
+Wire Wire Line
+	2210 2000 2390 2000
+Wire Wire Line
+	2070 2550 2390 2550
+Wire Wire Line
+	2820 1520 2820 2350
+Wire Wire Line
+	1550 1450 2210 1450
+Wire Wire Line
+	2210 1450 2210 2000
+Wire Wire Line
+	1550 1550 2070 1550
+Wire Wire Line
+	2070 1550 2070 2550
+Wire Wire Line
+	1550 1150 1790 1150
+Wire Wire Line
+	1550 1250 1790 1250
+Entry Wire Line
+	2720 1420 2820 1520
+Wire Wire Line
+	3010 1930 3010 1520
+Entry Wire Line
+	2910 1420 3010 1520
+Wire Bus Line
+	2910 1420 2660 1420
+Wire Bus Line
+	2660 1420 2660 620
+$Comp
+L TERM_06 TB1
+U 1 1 57E2236E
+P 1300 1400
+F 0 "TB1" H 1300 1780 50  0000 C CNN
+F 1 "TERM_06" H 1300 1020 50  0000 C CNN
+F 2 "" H 1300 200 50  0000 C CNN
+F 3 "" H 1300 200 50  0000 C CNN
+	1    1300 1400
+	1    0    0    -1
+$EndComp
+NoConn ~ 1550 1350
+NoConn ~ 1050 1350
 $EndSCHEMATC

Commit message: Updated schematic to include extra sheets.
Added several alternate wiring sheets and made some changes to the
schematic to reflect team decision. More to come.
Other:
- note added: "(Optional)"
Changed lines of the file:
@@
 $Descr USLetter 11000 8500
 encoding utf-8
-Sheet 3 4
+Sheet 3 6
 Title "District 1 Power Box"
-Date "2016-08-27"
-Rev "2"
+Date "2016-09-30"
+Rev "4"
 Comp "North Georgia Modurail"
 Comment1 ""
@@
 NoConn ~ 1550 1350
 NoConn ~ 1050 1350
+Text Notes 3930 3820 0    60   ~ 0
+(Optional)
 $EndSCHEMATC

Commit message: Updated schematic
Parts:
- removed M? (x2): M-Junction_Box, symbol M-Junction_Box_No-Tap
- removed TB1, TB2: TERM_06, symbol TERM_06
- added M-9A, M-9B: Anderson_PP9-M, symbol CONN_01X09
- added TB8: TERM_08, symbol TERM_08
- added TB?: TB4, symbol TBLOCK
- added TB? (x3): TBLOCK, symbol TBLOCK
- M?: value RRampmeter -> RRampMeter
Connections:
- net labels added: Black, Blue, Blue/Yellow, Brown, DCC_Ground, Gray, Green, Orange, Orange/Brown, Red, Red/Green, White, Yellow
- net labels removed: DCC-GROUND
- wire segments 117 -> 114
Other:
- note added: "LNRP Optional\non personal boxes."
- moved on the sheet: CB1
