File: KiCad Schematics/LEDs.sch (KiCad schematic (older format))
At the start: 12 parts

Commit message: Fixed LED wire assignments
All of the PSX-3s were wired differently from the PSX-4. This change
reflects the actual wiring, not the original intended wiring.
Connections:
- net Green_LED1+: now also D-R3.2 (A); no longer D-R1.2 (A)
- net Green_LED3+: now also D-R1.2 (A); no longer D-R3.2 (A)
- net Red_LED1-: now also LED-G3.1 (K), R3.1; no longer LED-G1.1 (K), R1.1
- net Red_LED3-: now also LED-G1.1 (K), R1.1; no longer LED-G3.1 (K), R3.1
Other:
- note added: "Note reverse colors\nfrom PSX-4"
Changed lines of the file:
@@
 $Descr USLetter 11000 8500
 encoding utf-8
-Sheet 15 16
+Sheet 9 16
 Title "NGM Power and LocoNet Power Boxes"
 Date "2016-10-08"
-Rev "5"
+Rev "5.1"
 Comp "North Georgia Modurail, Inc."
 Comment1 ""
@@
 AR Path="/57EBE249/57F943E9/57F7C962/57F7DB77" Ref="LED-R1"  Part="1"
 AR Path="/57F1B72E/57FA908E/57F7C962/57F7DB77" Ref="LED-R1"  Part="1"
+AR Path="/57EBE249/57F943E9/57F8CCA5/57F7DB77" Ref="LED-R1"  Part="1"
 F 0 "LED-R1" V 3460 2370 50  0000 C CNN
 F 1 "Track 1" V 3460 2950 79  0000 C CNN
@@
 AR Path="/57EBE249/57F943E9/57F7C962/57F7DB78" Ref="LED-R2"  Part="1"
 AR Path="/57F1B72E/57FA908E/57F7C962/57F7DB78" Ref="LED-R2"  Part="1"
+AR Path="/57EBE249/57F943E9/57F8CCA5/57F7DB78" Ref="LED-R2"  Part="1"
 F 0 "LED-R2" V 3450 3070 50  0000 C CNN
 F 1 "Track 2" V 3450 3670 79  0000 C CNN
@@
 AR Path="/57EBE249/57F943E9/57F7C962/57F7DB79" Ref="LED-R3"  Part="1"
 AR Path="/57F1B72E/57FA908E/57F7C962/57F7DB79" Ref="LED-R3"  Part="1"
+AR Path="/57EBE249/57F943E9/57F8CCA5/57F7DB79" Ref="LED-R3"  Part="1"
 F 0 "LED-R3" V 3450 3780 50  0000 C CNN
 F 1 "Track 3" V 3450 4360 79  0000 C CNN
@@
 AR Path="/57EBE249/57F943E9/57F7C962/57F7DB7A" Ref="LED-G1"  Part="1"
 AR Path="/57F1B72E/57FA908E/57F7C962/57F7DB7A" Ref="LED-G1"  Part="1"
+AR Path="/57EBE249/57F943E9/57F8CCA5/57F7DB7A" Ref="LED-G1"  Part="1"
 F 0 "LED-G1" V 4160 2360 50  0000 C CNN
 F 1 "LED" H 4160 2510 50  0001 C CNN
@@
 AR Path="/57EBE249/57F943E9/57F7C962/57F7DB7B" Ref="LED-G2"  Part="1"
 AR Path="/57F1B72E/57FA908E/57F7C962/57F7DB7B" Ref="LED-G2"  Part="1"
+AR Path="/57EBE249/57F943E9/57F8CCA5/57F7DB7B" Ref="LED-G2"  Part="1"
 F 0 "LED-G2" V 4160 3070 50  0000 C CNN
 F 1 "LED" H 4160 3220 50  0001 C CNN
@@
 AR Path="/57EBE249/57F943E9/57F7C962/57F7DB7C" Ref="LED-G3"  Part="1"
 AR Path="/57F1B72E/57FA908E/57F7C962/57F7DB7C" Ref="LED-G3"  Part="1"
+AR Path="/57EBE249/57F943E9/57F8CCA5/57F7DB7C" Ref="LED-G3"  Part="1"
 F 0 "LED-G3" V 4160 3760 50  0000 C CNN
 F 1 "LED" H 4160 3920 50  0001 C CNN
@@
 AR Path="/57EBE249/57F943E9/57F7C962/57F7DB7D" Ref="R4"  Part="1"
 AR Path="/57F1B72E/57FA908E/57F7C962/57F7DB7D" Ref="R4"  Part="1"
+AR Path="/57EBE249/57F943E9/57F8CCA5/57F7DB7D" Ref="R4"  Part="1"
 F 0 "R4" V 4910 5020 50  0000 C CNN
 F 1 "560 1/2W" V 4740 5020 39  0000 C CNN
@@
 AR Path="/57EBE249/57F943E9/57F7C962/57F7E3B1" Ref="LED-R4"  Part="1"
 AR Path="/57F1B72E/57FA908E/57F7C962/57F7E3B1" Ref="LED-R4"  Part="1"
+AR Path="/57EBE249/57F943E9/57F8CCA5/57F7E3B1" Ref="LED-R4"  Part="1"
 F 0 "LED-R4" V 3450 4540 50  0000 C CNN
 F 1 "Track 4" V 3450 5110 79  0000 C CNN
@@
 Text HLabel 3000 2360 0    60   Input ~ 0
 Red_LED1+
-Text Label 3060 2360 0    39   ~ 0
+Text Label 3030 3770 0    39   ~ 0
 Green
 Text Label 3040 3060 0    39   ~ 0
 Blue
-Text Label 3030 3770 0    39   ~ 0
+Text Label 3040 2360 0    39   ~ 0
 Orange
-Text Label 3020 4270 0    39   ~ 0
+Text Label 3040 2860 0    39   ~ 0
 Orange-White
 Text Label 3090 4520 0    39   ~ 0
 Brown
-Text Label 3060 2860 0    39   ~ 0
+Text Label 3030 4270 0    39   ~ 0
 Green-White
 Text Label 3020 5020 0    39   ~ 0
@@
 AR Path="/57EBE249/57F943E9/57F7C962/57F83F8C" Ref="LED-G4"  Part="1"
 AR Path="/57F1B72E/57FA908E/57F7C962/57F83F8C" Ref="LED-G4"  Part="1"
+AR Path="/57EBE249/57F943E9/57F8CCA5/57F83F8C" Ref="LED-G4"  Part="1"
 F 0 "LED-G4" V 4160 4510 50  0000 C CNN
 F 1 "LED" H 4160 4670 50  0001 C CNN
@@
 AR Path="/57EBE249/57F943E9/57F7C962/57F89882" Ref="R1"  Part="1"
 AR Path="/57F1B72E/57FA908E/57F7C962/57F89882" Ref="R1"  Part="1"
+AR Path="/57EBE249/57F943E9/57F8CCA5/57F89882" Ref="R1"  Part="1"
 F 0 "R1" V 4900 2860 50  0000 C CNN
 F 1 "560 1/2W" V 4730 2860 39  0000 C CNN
@@
 AR Path="/57EBE249/57F943E9/57F7C962/57F89A97" Ref="R2"  Part="1"
 AR Path="/57F1B72E/57FA908E/57F7C962/57F89A97" Ref="R2"  Part="1"
+AR Path="/57EBE249/57F943E9/57F8CCA5/57F89A97" Ref="R2"  Part="1"
 F 0 "R2" V 4910 3570 50  0000 C CNN
 F 1 "560 1/2W" V 4740 3570 39  0000 C CNN
@@
 AR Path="/57EBE249/57F943E9/57F7C962/57F89E27" Ref="R3"  Part="1"
 AR Path="/57F1B72E/57FA908E/57F7C962/57F89E27" Ref="R3"  Part="1"
+AR Path="/57EBE249/57F943E9/57F8CCA5/57F89E27" Ref="R3"  Part="1"
 F 0 "R3" V 4890 4270 50  0000 C CNN
 F 1 "560 1/2W" V 4720 4270 39  0000 C CNN
@@
 Wire Notes Line
 	1970 4430 5890 4430
+Text Notes 1040 3410 0    79   ~ 16
+Note reverse colors\nfrom PSX-4
 $EndSCHEMATC

Commit message: Updated schematic (reverted)
Reverted back to the correct wiring as the boards were rewired to spec.
Connections:
- net Green_LED1+: now also D-R1.2 (A); no longer D-R3.2 (A)
- net Green_LED3+: now also D-R3.2 (A); no longer D-R1.2 (A)
- net Red_LED1-: now also LED-G1.1 (K), R1.1; no longer LED-G3.1 (K), R3.1
- net Red_LED3-: now also LED-G3.1 (K), R3.1; no longer LED-G1.1 (K), R1.1
Other:
- note removed: "Note reverse colors\nfrom PSX-4"
Changed lines of the file:
@@
 $Descr USLetter 11000 8500
 encoding utf-8
-Sheet 9 16
+Sheet 5 16
 Title "NGM Power and LocoNet Power Boxes"
 Date "2016-10-08"
@@
 AR Path="/57F1B72E/57FA908E/57F7C962/57F7DB77" Ref="LED-R1"  Part="1"
 AR Path="/57EBE249/57F943E9/57F8CCA5/57F7DB77" Ref="LED-R1"  Part="1"
+AR Path="/57C1C56F/57F80E5A/57F8CCA5/57F7DB77" Ref="LED-R1"  Part="1"
 F 0 "LED-R1" V 3460 2370 50  0000 C CNN
 F 1 "Track 1" V 3460 2950 79  0000 C CNN
@@
 AR Path="/57F1B72E/57FA908E/57F7C962/57F7DB78" Ref="LED-R2"  Part="1"
 AR Path="/57EBE249/57F943E9/57F8CCA5/57F7DB78" Ref="LED-R2"  Part="1"
+AR Path="/57C1C56F/57F80E5A/57F8CCA5/57F7DB78" Ref="LED-R2"  Part="1"
 F 0 "LED-R2" V 3450 3070 50  0000 C CNN
 F 1 "Track 2" V 3450 3670 79  0000 C CNN
@@
 AR Path="/57F1B72E/57FA908E/57F7C962/57F7DB79" Ref="LED-R3"  Part="1"
 AR Path="/57EBE249/57F943E9/57F8CCA5/57F7DB79" Ref="LED-R3"  Part="1"
+AR Path="/57C1C56F/57F80E5A/57F8CCA5/57F7DB79" Ref="LED-R3"  Part="1"
 F 0 "LED-R3" V 3450 3780 50  0000 C CNN
 F 1 "Track 3" V 3450 4360 79  0000 C CNN
@@
 AR Path="/57F1B72E/57FA908E/57F7C962/57F7DB7A" Ref="LED-G1"  Part="1"
 AR Path="/57EBE249/57F943E9/57F8CCA5/57F7DB7A" Ref="LED-G1"  Part="1"
+AR Path="/57C1C56F/57F80E5A/57F8CCA5/57F7DB7A" Ref="LED-G1"  Part="1"
 F 0 "LED-G1" V 4160 2360 50  0000 C CNN
 F 1 "LED" H 4160 2510 50  0001 C CNN
@@
 AR Path="/57F1B72E/57FA908E/57F7C962/57F7DB7B" Ref="LED-G2"  Part="1"
 AR Path="/57EBE249/57F943E9/57F8CCA5/57F7DB7B" Ref="LED-G2"  Part="1"
+AR Path="/57C1C56F/57F80E5A/57F8CCA5/57F7DB7B" Ref="LED-G2"  Part="1"
 F 0 "LED-G2" V 4160 3070 50  0000 C CNN
 F 1 "LED" H 4160 3220 50  0001 C CNN
@@
 AR Path="/57F1B72E/57FA908E/57F7C962/57F7DB7C" Ref="LED-G3"  Part="1"
 AR Path="/57EBE249/57F943E9/57F8CCA5/57F7DB7C" Ref="LED-G3"  Part="1"
+AR Path="/57C1C56F/57F80E5A/57F8CCA5/57F7DB7C" Ref="LED-G3"  Part="1"
 F 0 "LED-G3" V 4160 3760 50  0000 C CNN
 F 1 "LED" H 4160 3920 50  0001 C CNN
@@
 AR Path="/57F1B72E/57FA908E/57F7C962/57F7DB7D" Ref="R4"  Part="1"
 AR Path="/57EBE249/57F943E9/57F8CCA5/57F7DB7D" Ref="R4"  Part="1"
+AR Path="/57C1C56F/57F80E5A/57F8CCA5/57F7DB7D" Ref="R4"  Part="1"
 F 0 "R4" V 4910 5020 50  0000 C CNN
 F 1 "560 1/2W" V 4740 5020 39  0000 C CNN
@@
 AR Path="/57F1B72E/57FA908E/57F7C962/57F7E3B1" Ref="LED-R4"  Part="1"
 AR Path="/57EBE249/57F943E9/57F8CCA5/57F7E3B1" Ref="LED-R4"  Part="1"
+AR Path="/57C1C56F/57F80E5A/57F8CCA5/57F7E3B1" Ref="LED-R4"  Part="1"
 F 0 "LED-R4" V 3450 4540 50  0000 C CNN
 F 1 "Track 4" V 3450 5110 79  0000 C CNN
@@
 Text HLabel 3000 2360 0    60   Input ~ 0
 Red_LED1+
-Text Label 3030 3770 0    39   ~ 0
+Text Label 3020 2360 0    39   ~ 0
 Green
 Text Label 3040 3060 0    39   ~ 0
 Blue
-Text Label 3040 2360 0    39   ~ 0
+Text Label 3020 3770 0    39   ~ 0
 Orange
-Text Label 3040 2860 0    39   ~ 0
+Text Label 3010 4270 0    39   ~ 0
 Orange-White
 Text Label 3090 4520 0    39   ~ 0
 Brown
-Text Label 3030 4270 0    39   ~ 0
+Text Label 3020 2860 0    39   ~ 0
 Green-White
 Text Label 3020 5020 0    39   ~ 0
@@
 AR Path="/57F1B72E/57FA908E/57F7C962/57F83F8C" Ref="LED-G4"  Part="1"
 AR Path="/57EBE249/57F943E9/57F8CCA5/57F83F8C" Ref="LED-G4"  Part="1"
+AR Path="/57C1C56F/57F80E5A/57F8CCA5/57F83F8C" Ref="LED-G4"  Part="1"
 F 0 "LED-G4" V 4160 4510 50  0000 C CNN
 F 1 "LED" H 4160 4670 50  0001 C CNN
@@
 AR Path="/57F1B72E/57FA908E/57F7C962/57F89882" Ref="R1"  Part="1"
 AR Path="/57EBE249/57F943E9/57F8CCA5/57F89882" Ref="R1"  Part="1"
+AR Path="/57C1C56F/57F80E5A/57F8CCA5/57F89882" Ref="R1"  Part="1"
 F 0 "R1" V 4900 2860 50  0000 C CNN
 F 1 "560 1/2W" V 4730 2860 39  0000 C CNN
@@
 AR Path="/57F1B72E/57FA908E/57F7C962/57F89A97" Ref="R2"  Part="1"
 AR Path="/57EBE249/57F943E9/57F8CCA5/57F89A97" Ref="R2"  Part="1"
+AR Path="/57C1C56F/57F80E5A/57F8CCA5/57F89A97" Ref="R2"  Part="1"
 F 0 "R2" V 4910 3570 50  0000 C CNN
 F 1 "560 1/2W" V 4740 3570 39  0000 C CNN
@@
 AR Path="/57F1B72E/57FA908E/57F7C962/57F89E27" Ref="R3"  Part="1"
 AR Path="/57EBE249/57F943E9/57F8CCA5/57F89E27" Ref="R3"  Part="1"
+AR Path="/57C1C56F/57F80E5A/57F8CCA5/57F89E27" Ref="R3"  Part="1"
 F 0 "R3" V 4890 4270 50  0000 C CNN
 F 1 "560 1/2W" V 4720 4270 39  0000 C CNN
@@
 Wire Notes Line
 	1970 4430 5890 4430
-Text Notes 1040 3410 0    79   ~ 16
-Note reverse colors\nfrom PSX-4
 $EndSCHEMATC

Commit message: Updated schematic to v5.2
Changed the green LED wiring to reflect common rail on pin J1-2 on PSX
units.
Connections:
- net Green_LED2- is gone; now on net Green_LED1-: R2.2
- net Green_LED3- is gone; now on net Green_LED1-: R1.2, R3.2
- net Green_LED1-: now also D-R3.1 (K)
- net Red_LED1-: no longer LED-G1.1 (K), R1.1
- net Red_LED2-: no longer LED-G2.1 (K), R2.1
- net Red_LED4-: no longer LED-G4.1 (K), R1.1
- net Red_LED3-: no longer names the net of LED-G3.1 (K), R3.1
- net Red_LED3-: no longer D-R3.1 (K)
- new net: LED-G1.1 (K), R1.1
- new net: LED-G2.1 (K), R2.1
- new net: LED-G4.1 (K), R1.1
Other:
- note added: "J2-1 Pins are common"
Changed lines of the file:
@@
 Title "NGM Power and LocoNet Power Boxes"
 Date "2016-10-08"
-Rev "5.1"
+Rev "5.2"
 Comp "North Georgia Modurail, Inc."
 Comment1 ""
@@
 Wire Wire Line
 	4160 4220 4160 4270
-Text HLabel 5140 2860 2    61   Input ~ 0
+Text HLabel 6710 5020 2    61   Input ~ 0
 Green_LED1-
 Text Label 4200 3070 0    39   ~ 0
@@
 Text Label 4200 3770 0    39   ~ 0
 Orange
-Text Label 4200 4270 0    39   ~ 0
+Text Label 5270 4270 0    39   ~ 0
 Orange-White
 Text Label 4210 4520 0    39   ~ 0
@@
 Wire Wire Line
 	4160 2860 4670 2860
-Text HLabel 5150 3570 2    61   Input ~ 0
-Green_LED2-
 Wire Wire Line
 	4160 3570 4680 3570
 Wire Wire Line
 	4160 4270 4660 4270
-Text HLabel 5140 4270 2    61   Input ~ 0
-Green_LED3-
 $Comp
 L R R1
@@
 	0    -1   -1   0
 $EndComp
-Wire Wire Line
-	4970 2860 5140 2860
 $Comp
 L R R2
@@
 	0    -1   -1   0
 $EndComp
-Wire Wire Line
-	5150 3570 4980 3570
 $Comp
 L R R3
@@
 $EndComp
 Wire Wire Line
-	5140 4270 4960 4270
-Wire Wire Line
 	4160 4970 4160 5020
 Wire Wire Line
 	4160 5020 4680 5020
-Text HLabel 5150 5020 2    61   Input ~ 0
-Green_LED3-
-Wire Wire Line
-	4980 5020 5150 5020
-Text Label 4190 5020 0    39   ~ 0
-Brown-White
-Text Label 4190 2860 0    39   ~ 0
-Green-White
-Text Label 4190 3570 0    39   ~ 0
-Blue-White
 Wire Notes Line
 	5890 4430 5890 5260
@@
 Wire Notes Line
 	1970 4430 5890 4430
+Wire Wire Line
+	4980 5020 6710 5020
+Wire Wire Line
+	4970 2860 6520 2860
+Wire Wire Line
+	6520 2860 6520 5020
+Connection ~ 6520 5020
+Wire Wire Line
+	4980 3570 6520 3570
+Connection ~ 6520 3570
+Wire Wire Line
+	4960 4270 6520 4270
+Connection ~ 6520 4270
+Text Notes 6740 4810 0    60   ~ 0
+J2-1 Pins are common
+Text Label 5270 3570 0    39   ~ 0
+Orange-White
+Text Label 5260 2860 0    39   ~ 0
+Orange-White
+Text Label 5280 5020 0    39   ~ 0
+Orange-White
 $EndSCHEMATC
