File: KiCad Schematics/Main Power Box.sch (KiCad schematic (older format))
At the start: 0 parts

Commit message: Simplified schematic
Added heirarchy sheets to simplify the schematic.
Parts:
- added C1: DCS-240, symbol TERM_07
- added C2: DB-200-2, symbol TERM_07_DB
- added C3: DB-200-1, symbol TERM_07_DB
- added CB1: 2A, symbol FUSE
- added LED1, LED2, LED3: LED, symbol LED
- added M1, M2: Fan, symbol Fan
- added P? (x2): Anderson_PP2, symbol CONN_01X02
- added P? (x2): TERM_12, symbol TERM_06
- added P? (x2): Anderson_PP9_M, symbol CONN_01X09
- added PS1: 19 VDC, symbol AHE220PS19
- added TB1: TERM_03, symbol TERM_03
- added TB2, TB3, TB5, TB6: TERM_06, symbol TERM_06
- added TB4, TB?: TERM_02, symbol TERM_02
- added TR1: TRANSFORMER_MCI_4-06-8016, symbol TRANSFORMER_MCI_4-06-8016
Connections:
- new net: TB1.1 (P1), TR1.10
- new net: TB1.2 (P2), TR1.6
- new net: CB1.1, TB1.2 (P2)
- new net: CB1.2, TB1.3 (P3)
- new net: M1.2 (-), M2.1 (+)
- new net: C2.3 (SYNC), C2.4 (GR)
- new net: C3.3 (SYNC), C3.4 (GR)
- new net 16VAC-B: TB1.1 (P1), TB4.1 (P1), TB4.2 (P2)
- new net 16VAC-W: TB1.3 (P3), TB?.1 (P1), TB?.2 (P2)
- new net Alarm1+: P?.1 (P1)
- new net Alarm1-: P?.2 (P2)
- new net Alarm2+: P?.3 (P3)
- new net Alarm2-: P?.4 (P4)
- new net Alarm3+: P?.5 (P5)
- new net Alarm3-: P?.6 (P6)
- new net Black: C1.2 (8A-), C2.2 (PWR), C3.2 (PWR), M2.2 (-), P?.2 (P2), P?.2 (P2), P?.8 (P8), P?.8 (P8), PS1.5 (-), TB3.3 (P3), TB3.4 (P4), TB4.2 (P2)
- new net Blue: C2.7 (RA), P?.4 (P4), TB5.2 (P2)
- new net Brown: P?.1 (P1)
- new net Gray: C1.4 (GR), C2.5 (GR), C3.5 (GR), P?.9 (P9), TB3.5 (P5), TB3.6 (P6)
- new net Green: C3.6 (RB), P?.5 (P5), TB5.1 (P1), TB5.3 (P3)
- new net LED1+: TB6.1 (P1)
- new net LED1-: TB6.2 (P2)
- new net LED2+: TB6.3 (P3)
- new net LED2-: TB6.4 (P4)
- new net LED3+: TB6.5 (P5)
- new net LED3-: TB6.6 (P6)
- new net Orange: P?.2 (P2)
- new net Red: C1.1 (8A+), C2.1 (PWR), C3.1 (PWR), C3.7 (RA), M1.1 (+), P?.1 (P1), P?.1 (P1), P?.6 (P6), PS1.4 (+), TB3.1 (P1), TB3.2 (P2), TB5.2 (P2), TB5.4 (P4)
- new net White: P?.7 (P7), P?.7 (P7), TB?.2 (P2)
- new net Yellow: C2.6 (RB), P?.3 (P3), TB5.1 (P1)
- no-connect marks 0 -> 16
Other:
- note added: "12 VDC fans\nin series"
- note added: "District 1\n(yard)"
- note added: "District 2\n(mainline)"

Commit message: Minor schematic changes
Parts:
- added SW1: DPDT, symbol DPDT
Connections:
- no-connect marks 16 -> 18
Other:
- note added: "RRampMeter\nSelection switch"
Changed lines of the file:
@@
 Text Notes 7240 4390 0    39   ~ 0
 District 1\n(yard)
+$Comp
+L DPDT SW1
+U 1 1 57F9AC42
+P 9130 1970
+F 0 "SW1" V 9070 1970 50  0000 C CNN
+F 1 "DPDT" V 8850 1970 50  0000 C CNN
+F 2 "" H 8505 2145 50  0000 C CNN
+F 3 "" H 8505 2145 50  0000 C CNN
+	1    9130 1970
+	0    -1   1    0
+$EndComp
+NoConn ~ 8930 2260
+NoConn ~ 9330 2260
+Text Notes 8890 1230 0    60   ~ 0
+RRampMeter\nSelection switch
 $EndSCHEMATC

Commit message: Updated schematic
Minor cleanup and update of PDF
Parts:
- removed SW1: DPDT, symbol DPDT
Connections:
- no-connect marks 18 -> 16
Other:
- note removed: "RRampMeter\nSelection switch"
Changed lines of the file:
@@
 Text Notes 7240 4390 0    39   ~ 0
 District 1\n(yard)
-$Comp
-L DPDT SW1
-U 1 1 57F9AC42
-P 9130 1970
-F 0 "SW1" V 9070 1970 50  0000 C CNN
-F 1 "DPDT" V 8850 1970 50  0000 C CNN
-F 2 "" H 8505 2145 50  0000 C CNN
-F 3 "" H 8505 2145 50  0000 C CNN
-	1    9130 1970
-	0    -1   1    0
-$EndComp
-NoConn ~ 8930 2260
-NoConn ~ 9330 2260
-Text Notes 8890 1230 0    60   ~ 0
-RRampMeter\nSelection switch
 $EndSCHEMATC
