File: KiCad Schematics/PSX-3.sch (KiCad schematic (older format))
At the start: 12 parts

Commit message: Fixed LED wire assignments
All of the PSX-3s were wired differently from the PSX-4. This change
reflects the actual wiring, not the original intended wiring.
Connections:
- net Rail_A: now also PSX?.J5-1 (LED+), PSX?.J5-2 (LED-); no longer PSX?.J5-1 (LED+), PSX?.J5-2 (LED-)
- net Track_3A: now also PSX?.J5-1 (LED+); no longer PSX?.J5-1 (LED+)
- net Track_3B: now also PSX?.J5-2 (LED-); no longer PSX?.J5-2 (LED-)
Other:
- note added: "CAT5\nPinout T568A"
- note added: "Note reverse\ncolors from\nPSX-4"
- note removed: "CAT5 (Type A)"
Changed lines of the file:
@@
 $Descr USLetter 11000 8500
 encoding utf-8
-Sheet 14 16
+Sheet 7 16
 Title "NGM Power and LocoNet Power Boxes"
 Date "2016-10-08"
-Rev "5"
+Rev "5.1"
 Comp "North Georgia Modurail, Inc."
 Comment1 ""
@@
 Text Label 3700 3400 3    60   ~ 0
 AlarmBus
-Text Label 1860 1700 0    39   ~ 0
+Text Label 1860 2200 0    39   ~ 0
 Orange
 Text Label 3230 2340 1    60   ~ 0
@@
 Text Label 3430 4040 0    60   ~ 0
 Red/Green
-Text Label 1870 2200 0    39   ~ 0
+Text Label 1870 1700 0    39   ~ 0
 Green
 Text Label 1860 1950 0    39   ~ 0
@@
 From Booster
 Text Notes 2110 770  0    79   ~ 0
-CAT5 (Type A)
+CAT5\nPinout T568A
 $Sheet
 S 860  1660 960  720
@@
 F7 "Red_LED3-" I R 1820 1800 39
 $EndSheet
-Text Label 1870 2300 0    39   ~ 0
+Text Label 1870 1800 0    39   ~ 0
 Green-White
 Text Label 1870 2050 0    39   ~ 0
 Blue-White
-Text Label 1850 1800 0    39   ~ 0
+Text Label 1860 2300 0    39   ~ 0
 Orange-White
 Text Label 2540 4330 0    60   ~ 0
@@
 Text Label 2540 4210 0    60   ~ 0
 Red
-Text Notes 1560 2560 0    79   ~ 0
-CAT5 (Type A)
+Text Notes 1570 2650 0    79   ~ 0
+CAT5\nPinout T568A
 Wire Wire Line
 	3230 3840 3230 3940
@@
 Wire Wire Line
 	2550 2300 1820 2300
+Text Notes 920  2020 0    39   ~ 0
+Note reverse\ncolors from\nPSX-4
 $EndSCHEMATC

Commit message: Updated schematic (reverted)
Reverted back to the correct wiring as the boards were rewired to spec.
Other:
- note removed: "Note reverse\ncolors from\nPSX-4"
Changed lines of the file:
@@
 $Descr USLetter 11000 8500
 encoding utf-8
-Sheet 7 16
+Sheet 3 16
 Title "NGM Power and LocoNet Power Boxes"
 Date "2016-10-08"
@@
 F1 "LEDs.sch" 60
 F2 "Red_LED2+" I R 1820 1950 39
-F3 "Red_LED1+" I R 1820 2200 39
-F4 "Red_LED3+" I R 1820 1700 39
-F5 "Red_LED1-" I R 1820 2300 39
+F3 "Red_LED1+" I R 1820 1700 39
+F4 "Red_LED3+" I R 1820 2200 39
+F5 "Red_LED1-" I R 1820 1800 39
 F6 "Red_LED2-" I R 1820 2050 39
-F7 "Red_LED3-" I R 1820 1800 39
+F7 "Red_LED3-" I R 1820 2300 39
 $EndSheet
 Text Label 1870 1800 0    39   ~ 0
@@
 Wire Wire Line
 	2550 2300 1820 2300
-Text Notes 920  2020 0    39   ~ 0
-Note reverse\ncolors from\nPSX-4
 $EndSCHEMATC

Commit message: Updated schematic to v5.2
Changed the green LED wiring to reflect common rail on pin J1-2 on PSX
units.
Connections:
- net Track_3B is gone; now on net Rail_A: PSX?.J2-1 (DCC2), PSX?.J5-2 (LED-), TB?.1 (P1)
- net Rail_A: now also PSX?.J2-1 (DCC2), TB?.1 (P1); no longer PSX?.J5-2 (LED-)
- removed net Track_2B: PSX?.J2-1 (DCC2), PSX?.J5-2 (LED-), TB?.1 (P1)
- new net Blue-White: PSX?.J5-2 (LED-)
- new net Green-White: PSX?.J5-2 (LED-)
Other:
- note added: "J2-1 Pins are common"
Changed lines of the file:
@@
 Title "NGM Power and LocoNet Power Boxes"
 Date "2016-10-08"
-Rev "5.1"
+Rev "5.2"
 Comp "North Georgia Modurail, Inc."
 Comment1 ""
@@
 F3 "Green_LED2+" I R 1800 1050 39
 F4 "Green_LED3+" I R 1800 1250 39
-F5 "Green_LED1-" I R 1800 950 39
-F6 "Green_LED2-" I R 1800 1150 39
-F7 "Green_LED3-" I R 1800 1350 39
+F5 "Green_LED1-" I R 1800 1350 39
 $EndSheet
 Text HLabel 2410 4210 0    60   Input ~ 0
@@
 	5050 2780 4950 2780
 Wire Wire Line
-	5610 1350 5610 2410
+	5610 950  5610 2410
 Wire Wire Line
 	5510 2410 5510 1250
@@
 	1800 1250 7110 1250
 Wire Wire Line
-	4470 1150 4470 2410
+	4470 1350 4470 2410
 Wire Wire Line
 	4370 2410 4370 1050
 Wire Wire Line
 	1800 1050 7110 1050
-Wire Wire Line
-	3330 950  3330 2410
 Wire Wire Line
 	3230 2410 3230 850
@@
 Connection ~ 5510 1250
 Wire Wire Line
-	1800 950  7110 950
-Wire Wire Line
-	1800 1150 7110 1150
-Wire Wire Line
 	1800 1350 7110 1350
 Wire Wire Line
@@
 Wire Wire Line
 	8530 1350 7610 1350
-Connection ~ 3330 950
-Connection ~ 4470 1150
 Connection ~ 5610 1350
-Text Label 1850 950  0    39   ~ 0
-Green-White
-Text Label 1850 1150 0    39   ~ 0
-Blue-White
 Text Label 1850 1350 0    39   ~ 0
 Orange-White
@@
 Wire Wire Line
 	2550 2300 1820 2300
+Connection ~ 4470 1350
+Connection ~ 3330 1350
+Wire Wire Line
+	3330 1350 3330 2410
+Wire Wire Line
+	7110 950  5610 950
+Wire Wire Line
+	7110 1150 5610 1150
+Connection ~ 5610 1150
+Text Notes 5730 2390 0    60   ~ 0
+J2-1 Pins are common
 $EndSCHEMATC

Commit message: Update schematic
Connections:
- net at PSX?.1 (+): now also B2.2
- net at PSX?.2 (-): now also B2.1
- net at PSX?.1 (+): now also B3.2
- net at PSX?.2 (-): now also B3.1
- net at PSX?.1 (+): now also B1.2
- net at PSX?.2 (-): now also B1.1
Other:
- moved on the sheet: B1, B2, B3
Changed lines of the file:
@@
 $Descr USLetter 11000 8500
 encoding utf-8
-Sheet 14 16
+Sheet 3 16
 Title "NGM Power and LocoNet Power Boxes"
 Date "2016-10-08"
@@
 NoConn ~ 5510 3840
 NoConn ~ 5610 3840
-Entry Wire Line
-	3600 3200 3700 3300
-Entry Wire Line
-	3600 3300 3700 3400
-Entry Wire Line
-	4730 3200 4830 3300
-Entry Wire Line
-	4730 3300 4830 3400
-Entry Wire Line
-	5870 3300 5970 3400
-Entry Wire Line
-	5870 3200 5970 3300
-Text Label 5970 3400 3    60   ~ 0
-AlarmBus
-Text Label 4830 3400 3    60   ~ 0
-AlarmBus
-Text Label 3700 3400 3    60   ~ 0
-AlarmBus
 Text Label 1860 2200 0    39   ~ 0
 Orange
@@
 L Crystal_Small B1
 U 1 1 57F85365
-P 5640 5130
+P 3700 3200
 AR Path="/57EBE249/57F943E9/57F85365" Ref="B1"  Part="1"
 AR Path="/57C1C56F/57F80E5A/57F85365" Ref="B1"  Part="1"
 AR Path="/57F1B72E/57FA908E/57F85365" Ref="B1"  Part="1"
-F 0 "B1" H 5640 5230 50  0000 C CNN
-F 1 "Piezo" H 5640 5030 50  0001 C CNN
-F 2 "" H 5640 5130 50  0000 C CNN
-F 3 "" H 5640 5130 50  0000 C CNN
-	1    5640 5130
+F 0 "B1" H 3700 3300 50  0000 C CNN
+F 1 "Piezo" H 3700 3100 50  0001 C CNN
+F 2 "" H 3700 3200 50  0000 C CNN
+F 3 "" H 3700 3200 50  0000 C CNN
+	1    3700 3200
 	1    0    0    -1
 $EndComp
@@
 L Crystal_Small B2
 U 1 1 57F8557A
-P 5640 5370
+P 4830 3200
 AR Path="/57EBE249/57F943E9/57F8557A" Ref="B2"  Part="1"
 AR Path="/57C1C56F/57F80E5A/57F8557A" Ref="B2"  Part="1"
 AR Path="/57F1B72E/57FA908E/57F8557A" Ref="B2"  Part="1"
-F 0 "B2" H 5640 5470 50  0000 C CNN
-F 1 "Piezo" H 5640 5270 50  0001 C CNN
-F 2 "" H 5640 5370 50  0000 C CNN
-F 3 "" H 5640 5370 50  0000 C CNN
-	1    5640 5370
+F 0 "B2" H 4830 3300 50  0000 C CNN
+F 1 "Piezo" H 4830 3100 50  0001 C CNN
+F 2 "" H 4830 3200 50  0000 C CNN
+F 3 "" H 4830 3200 50  0000 C CNN
+	1    4830 3200
 	1    0    0    -1
 $EndComp
@@
 L Crystal_Small B3
 U 1 1 57F855A1
-P 5640 5620
+P 5970 3200
 AR Path="/57EBE249/57F943E9/57F855A1" Ref="B3"  Part="1"
 AR Path="/57C1C56F/57F80E5A/57F855A1" Ref="B3"  Part="1"
 AR Path="/57F1B72E/57FA908E/57F855A1" Ref="B3"  Part="1"
-F 0 "B3" H 5640 5720 50  0000 C CNN
-F 1 "Piezo" H 5640 5520 50  0001 C CNN
-F 2 "" H 5640 5620 50  0000 C CNN
-F 3 "" H 5640 5620 50  0000 C CNN
-	1    5640 5620
-	1    0    0    -1
-$EndComp
-Entry Wire Line
-	5870 5130 5970 5030
-Entry Wire Line
-	5870 5370 5970 5270
-Entry Wire Line
-	5870 5620 5970 5520
-Entry Wire Line
-	5300 5230 5400 5130
-Entry Wire Line
-	5300 5470 5400 5370
-Entry Wire Line
-	5300 5720 5400 5620
+F 0 "B3" H 5970 3300 50  0000 C CNN
+F 1 "Piezo" H 5970 3100 50  0001 C CNN
+F 2 "" H 5970 3200 50  0000 C CNN
+F 3 "" H 5970 3200 50  0000 C CNN
+	1    5970 3200
+	1    0    0    -1
+$EndComp
 Text HLabel 8530 850  2    60   Input ~ 0
 Track_1A
@@
 	3490 3200 3600 3200
 Wire Wire Line
-	3490 3300 3600 3300
-Wire Wire Line
 	4630 3200 4730 3200
 Wire Wire Line
-	4630 3300 4730 3300
-Wire Wire Line
 	5770 3200 5870 3200
 Wire Wire Line
-	5770 3300 5870 3300
-Wire Bus Line
-	3700 3300 3700 3600
-Wire Bus Line
-	4830 3300 4830 3600
+	5770 3300 6140 3300
 Wire Wire Line
 	2550 2880 2770 2880
@@
 	3130 4330 2420 4330
 Wire Wire Line
-	5870 5620 5740 5620
-Wire Wire Line
-	5740 5370 5870 5370
-Wire Wire Line
-	5870 5130 5740 5130
-Wire Wire Line
-	5540 5130 5400 5130
-Wire Wire Line
-	5540 5370 5400 5370
-Wire Wire Line
-	5540 5620 5400 5620
-Wire Bus Line
-	5300 5230 5300 5860
-Wire Bus Line
-	5300 5860 5970 5860
-Wire Bus Line
-	5970 5860 5970 3300
-Wire Wire Line
 	7610 850  8530 850
 Wire Wire Line
@@
 Text Notes 5730 2390 0    60   ~ 0
 J2-1 Pins are common
+Wire Wire Line
+	6070 3200 6140 3200
+Wire Wire Line
+	6140 3200 6140 3300
+Wire Wire Line
+	3490 3300 3850 3300
+Wire Wire Line
+	3850 3300 3850 3200
+Wire Wire Line
+	3850 3200 3800 3200
+Wire Wire Line
+	4630 3300 5000 3300
+Wire Wire Line
+	5000 3300 5000 3200
+Wire Wire Line
+	5000 3200 4930 3200
 $EndSCHEMATC
